Commit message: Reorganized directory structure.

File: robot_description/urdf/generic_roomba_bot.urdf.xacro (robot description, xacro)
@@ -11,5 +11,5 @@
     <xacro:property name="wheel_width" default="0.05" />
     <xacro:property name="wheel_sep" value="${2*0.9*bot_radius}" />
-    <xacro:include filename="$(find ros2_robot_sims)/urdf/generic_roomba_bot_gazebo.urdf.xacro" />
+    <xacro:include filename="$(find robot_description)/urdf/generic_roomba_bot_gazebo.urdf.xacro" />
     <link name="base_link">
         <inertial>
@@ -60,5 +60,5 @@
         <parent link="base_link" />
         <child link="left_wheel" />
-        <origin xyz="0 -${wheel_sep/2} 0" rpy="1.5707 0 0" />
+        <origin xyz="0 ${wheel_sep/2} 0" rpy="1.5707 0 0" />
         <axis xyz="0 0 1" />
     </joint>
@@ -83,5 +83,5 @@
         <parent link="base_link" />
         <child link="right_wheel" />
-        <origin xyz="0 ${wheel_sep/2} 0" rpy="1.5707 0 0" />
+        <origin xyz="0 -${wheel_sep/2} 0" rpy="1.5707 0 0" />
         <axis xyz="0 0 1" />
     </joint>
@@ -148,5 +148,5 @@
     </link>
     <!-- Diff drive plugin -->
-    <xacro:include filename="$(find ros2_robot_sims)/urdf/diff_drive_plugin.urdf.xacro" />
+    <xacro:include filename="$(find robot_description)/urdf/diff_drive_plugin.urdf.xacro" />
     <xacro:diff_drive_plugin namespace="" update_rate="10" left_joint="base_link2left_wheel" right_joint="base_link2right_wheel" wheel_sep="${wheel_sep}" wheel_diam="${2*wheel_radius}" wheel_acc="1.0" wheel_torq="20" />
     <!-- 3-D LiDAR -->
@@ -155,3 +155,9 @@
         <origin xyz="0 0 ${top_length}" rpy="0 0 0" />
     </xacro:VLP-16>
+    <!-- P3D plugin -->
+    <xacro:include filename="$(find robot_description)/urdf/p3d_plugin.urdf.xacro"/>
+    <xacro:p3d_plugin namespace="" link_name="base_link" frame_name="map">
+        <xyz_offsets>0 0 0</xyz_offsets>
+        <rpy_offsets>0 0 0</rpy_offsets>
+    </xacro:p3d_plugin>
 </robot>

Commit message: Modified some default values.

File: robot_description/urdf/generic_roomba_bot.urdf.xacro (robot description, xacro)
@@ -2,6 +2,6 @@
 <robot xmlns:xacro="http://www.ros.org/wiki/xacro" name="generic_roomba_bot">
     <xacro:property name="bot_mass" default="25.0" />
-    <xacro:property name="bot_radius" default="0.75" />
-    <xacro:property name="bot_length" default="1.5" />
+    <xacro:property name="bot_radius" default="0.5" />
+    <xacro:property name="bot_length" default="1.0" />
     <xacro:property name="top_mass" value="${0.1*bot_mass}" />
     <xacro:property name="top_radius" value="${0.15*bot_radius}" />
@@ -10,5 +10,5 @@
     <xacro:property name="wheel_radius" default="0.2" />
     <xacro:property name="wheel_width" default="0.05" />
-    <xacro:property name="wheel_sep" value="${2*0.9*bot_radius}" />
+    <xacro:property name="wheel_sep" value="${2*0.8*bot_radius}" />
     <xacro:include filename="$(find robot_description)/urdf/generic_roomba_bot_gazebo.urdf.xacro" />
     <link name="base_link">

Commit message: 1. Added python utilities. 2. Added rosbag2 record and play launch files. 3. Corrected generic_roomba_bot travel direction.

File: robot_description/urdf/generic_roomba_bot.urdf.xacro (robot description, xacro)
@@ -60,5 +60,5 @@
         <parent link="base_link" />
         <child link="left_wheel" />
-        <origin xyz="0 ${wheel_sep/2} 0" rpy="1.5707 0 0" />
+        <origin xyz="0 ${wheel_sep/2} 0" rpy="-1.5707 0 0" />
         <axis xyz="0 0 1" />
     </joint>
@@ -83,5 +83,5 @@
         <parent link="base_link" />
         <child link="right_wheel" />
-        <origin xyz="0 -${wheel_sep/2} 0" rpy="1.5707 0 0" />
+        <origin xyz="0 -${wheel_sep/2} 0" rpy="-1.5707 0 0" />
         <axis xyz="0 0 1" />
     </joint>
